Commit message: added ros joints mimic plugin

File: yahboomcar_description/urdf/yahboomcar_X3plus.gazebo.xacro (robot description, xacro)
@@ -1,8 +1,25 @@
 <?xml version="1.0"?>
 <robot name="yahboomcar_X3plus" xmlns:xacro="http://www.ros.org/wiki/xacro">
+<xacro:macro name="mimic_joint_plugin_gazebo" params="name_prefix parent_joint mimic_joint has_pid:=false multiplier:=1.0 offset:=0 sensitiveness:=0.0 max_effort:=1.0 robot_namespace:=''">
+    <gazebo>
+	    <plugin name="${name_prefix}mimic_joint_plugin" filename="libroboticsgroup_gazebo_mimic_joint_plugin.so">
+		    <joint>${parent_joint}</joint>
+			<mimicJoint>${mimic_joint}</mimicJoint>
+			<xacro:if value="${has_pid}">                     <!-- if set to true, PID parameters from "/gazebo_ros_control/pid_gains/${mimic_joint}" are loaded -->
+			    <hasPID />
+			</xacro:if>
+			<multiplier>${multiplier}</multiplier>
+			<offset>${offset}</offset>
+			<sensitiveness>${sensitiveness}</sensitiveness>   <!-- if absolute difference between setpoint and process value is below this threshold, do nothing; 0.0 = disable [rad] -->
+			<maxEffort>${max_effort}</maxEffort>              <!-- only taken into account if has_pid:=true [Nm] -->
+			<xacro:unless value="${robot_namespace == ''}">
+			<robotNamespace>${robot_namespace}</robotNamespace>
+			</xacro:unless>
+		</plugin>
+	</gazebo>
+</xacro:macro>
 <xacro:property name="camera_name"  value  = "mycamera"/>
 <xacro:property name="frame_name"  value  = "camera_link"/>
 <gazebo reference="camera_link">
-    <!--arg name="camera_name"  default  = "mycamera"/-->
     <sensor name="astra_camera" type="depth">
         <visualize>true</visualize>
@@ -88,5 +105,5 @@
 </gazebo>
   <!-- ROS2 CONTROL -->
-    <ros2_control name="GazeboSystem" type="system">
+    <ros2_control name="yahboomcar_x3plusSystem" type="system">
     <hardware>
       <plugin>gazebo_ros2_control/GazeboSystem</plugin>
@@ -97,4 +114,12 @@
         <param name="max">6.28</param>
       </command_interface>
+      <command_interface name="velocity">
+          <param name="min">-1</param>
+          <param name="max">1</param>
+      </command_interface>
+      <command_interface name="effort">
+          <param name="min">-1000</param>
+          <param name="max">1000</param>
+      </command_interface>
       <state_interface name="position"/>
       <state_interface name="velocity"/>
@@ -106,4 +131,12 @@
         <param name="max">6.28</param>
       </command_interface>
+      <command_interface name="velocity">
+          <param name="min">-1</param>
+          <param name="max">1</param>
+      </command_interface>
+      <command_interface name="effort">
+          <param name="min">-1000</param>
+          <param name="max">1000</param>
+      </command_interface>
       <state_interface name="position"/>
       <state_interface name="velocity"/>
@@ -115,4 +148,12 @@
         <param name="max">6.28</param>
       </command_interface>
+      <command_interface name="velocity">
+          <param name="min">-1</param>
+          <param name="max">1</param>
+      </command_interface>
+      <command_interface name="effort">
+          <param name="min">-1000</param>
+          <param name="max">1000</param>
+      </command_interface>
       <state_interface name="position"/>
       <state_interface name="velocity"/>
@@ -124,4 +165,12 @@
         <param name="max">6.28</param>
       </command_interface>
+      <command_interface name="velocity">
+          <param name="min">-1</param>
+          <param name="max">1</param>
+      </command_interface>
+      <command_interface name="effort">
+          <param name="min">-1000</param>
+          <param name="max">1000</param>
+      </command_interface>
       <state_interface name="position"/>
       <state_interface name="velocity"/>
@@ -133,4 +182,12 @@
         <param name="max">6.28</param>
       </command_interface>
+      <command_interface name="velocity">
+          <param name="min">-1</param>
+          <param name="max">1</param>
+      </command_interface>
+      <command_interface name="effort">
+          <param name="min">-1000</param>
+          <param name="max">1000</param>
+      </command_interface>
       <state_interface name="position"/>
       <state_interface name="velocity"/>
@@ -141,4 +198,97 @@
         <param name="min">-6.28</param>
         <param name="max">6.28</param>
+      </command_interface>
+      <command_interface name="velocity">
+          <param name="min">-1</param>
+          <param name="max">1</param>
+      </command_interface>
+      <command_interface name="effort">
+          <param name="min">-1000</param>
+          <param name="max">1000</param>
+      </command_interface>
+      <state_interface name="position"/>
+      <state_interface name="velocity"/>
+      <state_interface name="effort"/>
+    </joint>
+    <joint name="rlink_joint2_mimic">
+      <command_interface name="position">
+        <param name="min">-6.28</param>
+        <param name="max">6.28</param>
+      </command_interface>
+      <command_interface name="velocity">
+          <param name="min">-1</param>
+          <param name="max">1</param>
+      </command_interface>
+      <command_interface name="effort">
+          <param name="min">-1000</param>
+          <param name="max">1000</param>
+      </command_interface>
+      <state_interface name="position"/>
+      <state_interface name="velocity"/>
+      <state_interface name="effort"/>
+    </joint>
+    <joint name="rlink_joint3_mimic">
+      <command_interface name="position">
+        <param name="min">-6.28</param>
+        <param name="max">6.28</param>
+      </command_interface>
+      <command_interface name="velocity">
+          <param name="min">-1</param>
+          <param name="max">1</param>
+      </command_interface>
+      <command_interface name="effort">
+          <param name="min">-1000</param>
+          <param name="max">1000</param>
+      </command_interface>
+      <state_interface name="position"/>
+      <state_interface name="velocity"/>
+      <state_interface name="effort"/>
+    </joint>
+    <joint name="llink_joint1_mimic">
+      <command_interface name="position">
+        <param name="min">-6.28</param>
+        <param name="max">6.28</param>
+      </command_interface>
+      <command_interface name="velocity">
+          <param name="min">-1</param>
+          <param name="max">1</param>
+      </command_interface>
+      <command_interface name="effort">
+          <param name="min">-1000</param>
+          <param name="max">1000</param>
+      </command_interface>
+      <state_interface name="position"/>
+      <state_interface name="velocity"/>
+      <state_interface name="effort"/>
+    </joint>
+    <joint name="llink_joint2_mimic">
+      <command_interface name="position">
+        <param name="min">-6.28</param>
+        <param name="max">6.28</param>
+      </command_interface>
+      <command_interface name="velocity">
+          <param name="min">-1</param>
+          <param name="max">1</param>
+      </command_interface>
+      <command_interface name="effort">
+          <param name="min">-1000</param>
+          <param name="max">1000</param>
+      </command_interface>
+      <state_interface name="position"/>
+      <state_interface name="velocity"/>
+      <state_interface name="effort"/>
+    </joint>
+    <joint name="llink_joint3_mimic">
+      <command_interface name="position">
+        <param name="min">-6.28</param>
+        <param name="max">6.28</param>
+      </command_interface>
+      <command_interface name="velocity">
+          <param name="min">-1</param>
+          <param name="max">1</param>
+      </command_interface>
+      <command_interface name="effort">
+          <param name="min">-1000</param>
+          <param name="max">1000</param>
       </command_interface>
       <state_interface name="position"/>
@@ -149,5 +299,5 @@
   <gazebo>
     <plugin filename="libgazebo_ros2_control.so" name="gazebo_ros2_control">
-      <parameters>$(find yahboomcar_control)/config/position_controller.yaml</parameters>
+      <parameters>$(find yahboomcar_control)/config/joint_trajectory_controller.yaml</parameters>
     </plugin>
   </gazebo>

File: yahboomcar_description/urdf/yahboomcar_X3plus.urdf.xacro (robot description, xacro)
@@ -8,5 +8,4 @@
         <color rgba="0.7 0.7 0.7 1"/>
     </material>
-    <link name="base_footprint"/>
     <!-- common link / base_link -->
     <xacro:macro name="common_link" params="name material path *origin">
@@ -27,5 +26,5 @@
     </xacro:macro>
     <!-- revolute joint-->
-    <xacro:macro name="revolute_joint" params="name parent child xyz rpy axisZ lower upper">
+    <xacro:macro name="revolute_joint" params="name parent child xyz rpy axisZ lower upper vel">
         <joint name="${name}" type="revolute">
             <parent link="${parent}"/>
@@ -33,5 +32,5 @@
             <origin xyz="${xyz}" rpy="${rpy}"/>
             <axis xyz="0 0 ${axisZ}"/>
-            <limit lower="${lower}" upper="${upper}" effort="100" velocity="1"/>
+            <limit lower="${lower}" upper="${upper}" effort="100" velocity="${vel}"/>
         </joint>
     </xacro:macro>
@@ -164,20 +163,29 @@
     </xacro:common_link>
     <!-- END RGBD Camera Links -->
+    <!-- classic world joint -->
+    <link name="world" />
     <!-- joint concatenation -->
-    <xacro:fixed_joint name="base_joint" parent="base_footprint" child="base_link" xyz="0.0 0.0 0.076" rpy="0 0 0"/>
-    <xacro:revolute_joint name="arm_joint1" parent="base_link" child="arm_link1" xyz="0 0 0.07" rpy="0 0 ${pi/2}" axisZ="-1" lower="-${pi/2}" upper="${pi/2}"/>
-    <xacro:revolute_joint name="arm_joint2" parent="arm_link1" child="arm_link2" xyz="0 0 0.0405" rpy="-${pi/2} 0 0" axisZ="-1" lower="-${pi/2}" upper="${pi/2}"/>
-    <xacro:revolute_joint name="arm_joint3" parent="arm_link2" child="arm_link3" xyz="0 -0.0829 0" rpy="0 0 0" axisZ="-1" lower="-${pi/2}" upper="${pi/2}"/>
-    <xacro:revolute_joint name="arm_joint4" parent="arm_link3" child="arm_link4" xyz="0 -0.0829 0" rpy="0 0 0" axisZ="-1" lower="-${pi/2}" upper="${pi/2}"/>
-    <xacro:revolute_joint name="arm_joint5" parent="arm_link4" child="arm_link5" xyz="-0.00215 -0.17455 0" rpy="${pi/2} 0 0" axisZ="1" lower="-${pi/2}" upper="${pi}"/>
-    <xacro:revolute_joint name="grip_joint" parent="arm_link5" child="rlink1" xyz="-0.0035 -0.012625 -0.0685" rpy="0 -${pi/2} 0" axisZ="1" lower="-${pi/2}" upper="0"/>
+    <xacro:fixed_joint name="base_joint" parent="world" child="base_link" xyz="0.0 0.0 0.076" rpy="0 0 0"/>
+    <xacro:revolute_joint name="arm_joint1" parent="base_link" child="arm_link1" xyz="0 0 0.07" rpy="0 0 ${pi/2}" axisZ="-1" lower="-${pi/2}" upper="${pi/2}" vel="3.14"/>
+    <xacro:revolute_joint name="arm_joint2" parent="arm_link1" child="arm_link2" xyz="0 0 0.0405" rpy="-${pi/2} 0 0" axisZ="-1" lower="-${pi/2}" upper="${pi/2}" vel="3.14"/>
+    <xacro:revolute_joint name="arm_joint3" parent="arm_link2" child="arm_link3" xyz="0 -0.0829 0" rpy="0 0 0" axisZ="-1" lower="-${pi/2}" upper="${pi/2}" vel="3.14"/>
+    <xacro:revolute_joint name="arm_joint4" parent="arm_link3" child="arm_link4" xyz="0 -0.0829 0" rpy="0 0 0" axisZ="-1" lower="-${pi/2}" upper="${pi/2}" vel="3.14"/>
+    <xacro:revolute_joint name="arm_joint5" parent="arm_link4" child="arm_link5" xyz="-0.00215 -0.17455 0" rpy="${pi/2} 0 0" axisZ="1" lower="-${pi/2}" upper="${pi}" vel="3.14"/>
+    <xacro:revolute_joint name="grip_joint" parent="arm_link5" child="rlink1" xyz="-0.0035 -0.012625 -0.0685" rpy="0 -${pi/2} 0" axisZ="1" lower="-${pi/2}" upper="0" vel="3.14"/>
     <!-- END joint concatenation -->
     <!-- gripper joints -->
-    <xacro:continuous_joint name="rlink_joint2" parent="rlink1" child="rlink2" xyz="0.03 -0.00075429 0" rpy="0 0 0" mimic="-1"/>
-    <xacro:continuous_joint name="rlink_joint3" parent="arm_link5" child="rlink3" xyz="-0.0035 -0.0045 -0.0505" rpy="0 -${pi/2} 0" mimic="1"/>
-    <xacro:continuous_joint name="llink_joint1" parent="arm_link5" child="llink1" xyz="-0.0035 0.012375 -0.0685" rpy="0 -${pi/2} 0" mimic="-1"/>
-    <xacro:continuous_joint name="llink_joint2" parent="llink1" child="llink2" xyz="0.03 0.00065104 0" rpy="0 0 0" mimic="1"/>
-    <xacro:continuous_joint name="llink_joint3" parent="arm_link5" child="llink3" xyz="-0.0035 0.0045 -0.0505" rpy="0 -${pi/2} 0" mimic="-1"/>
+    <xacro:continuous_joint name="rlink_joint2_mimic" parent="rlink1" child="rlink2" xyz="0.03 -0.00075429 0" rpy="0 0 0" mimic="-1"/>
+    <xacro:continuous_joint name="rlink_joint3_mimic" parent="arm_link5" child="rlink3" xyz="-0.0035 -0.0045 -0.0505" rpy="0 -${pi/2} 0" mimic="1"/>
+    <xacro:continuous_joint name="llink_joint1_mimic" parent="arm_link5" child="llink1" xyz="-0.0035 0.012375 -0.0685" rpy="0 -${pi/2} 0" mimic="-1"/>
+    <xacro:continuous_joint name="llink_joint2_mimic" parent="llink1" child="llink2" xyz="0.03 0.00065104 0" rpy="0 0 0" mimic="1"/>
+    <xacro:continuous_joint name="llink_joint3_mimic" parent="arm_link5" child="llink3" xyz="-0.0035 0.0045 -0.0505" rpy="0 -${pi/2} 0" mimic="-1"/>
     <!-- END gripper joints -->
+    <!-- Gripper Mimic -->
+    <xacro:mimic_joint_plugin_gazebo name_prefix="rlink_join2_mimic" parent_joint="gripper_joint" mimic_joint="rlink_joint2_mimic" has_pid="false" multiplier="-1" max_effort="10.6" />
+    <xacro:mimic_joint_plugin_gazebo name_prefix="rlink_join3_mimic" parent_joint="gripper_joint" mimic_joint="rlink_joint3_mimic" has_pid="false" multiplier="1" max_effort="10.6" />
+    <xacro:mimic_joint_plugin_gazebo name_prefix="llink_join1_mimic" parent_joint="gripper_joint" mimic_joint="llink_joint1_mimic" has_pid="false" multiplier="-1" max_effort="10.6" />
+    <xacro:mimic_joint_plugin_gazebo name_prefix="llink_join2_mimic" parent_joint="gripper_joint" mimic_joint="llink_joint2_mimic" has_pid="false" multiplier="1" max_effort="10.6" />
+    <xacro:mimic_joint_plugin_gazebo name_prefix="llink_join3_mimic" parent_joint="gripper_joint" mimic_joint="llink_joint3_mimic" has_pid="false" multiplier="-1" max_effort="10.6" />
+    <!-- END of Joint Mimic -->
     <!--rgb camera joint -->
     <xacro:fixed_joint name="mono_joint" parent="arm_link4" child="mono_link" xyz="-0.0481 -0.05145 -0.0022" rpy="${pi/2} 0 0"/>
@@ -233,4 +241,5 @@
     <kd>1000000</kd>
     <material>Gazebo/Green</material>
+    <selfCollide>false</selfCollide>
   </gazebo>
   <gazebo reference="rlink2">
@@ -240,4 +249,5 @@
     <kd>1000000</kd>
     <material>Gazebo/Green</material>
+    <selfCollide>false</selfCollide>
   </gazebo>
   <gazebo reference="rlink3">
@@ -247,4 +257,5 @@
     <kd>1000000</kd>
     <material>Gazebo/Green</material>
+    <selfCollide>false</selfCollide>
   </gazebo>
   <gazebo reference="llink1">
@@ -254,4 +265,5 @@
     <kd>1000000</kd>
     <material>Gazebo/Green</material>
+    <selfCollide>false</selfCollide>
   </gazebo>
   <gazebo reference="llink2">
@@ -261,4 +273,5 @@
     <kd>1000000</kd>
     <material>Gazebo/Green</material>
+    <selfCollide>false</selfCollide>
   </gazebo>
   <gazebo reference="llink3">
@@ -268,4 +281,5 @@
     <kd>1000000</kd>
     <material>Gazebo/Green</material>
+    <selfCollide>false</selfCollide>
   </gazebo>
   <gazebo reference="mono_link">
